File: TemperatureLogger/TemperatureLogger.kicad_sch (KiCad schematic)
At the start: 43 parts, among them J1 OUTPUT, J2 OUTPUT, J3 USB_C_Receptacle_USB2.0, J4 Conn_02x03_Odd_Even, J5 Conn_02x03_Odd_Even, K1 G6E, K2 G6E, Q1 BC847C, Q2 BC847C, U1 STM32F072C8Tx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

Commit message: added external flash and corrected issue with output disable for digital isolators
Parts:
- added C60: 100n, Capacitor_SMD:C_0603_1608Metric, symbol Device:C_Small
- added D5: LED_RED, LED_SMD:LED_0603_1608Metric, symbol Device:LED
- added D6: LED_GREEN, LED_SMD:LED_0603_1608Metric, symbol Device:LED
- added R20, R21: 620, Resistor_SMD:R_0603_1608Metric, symbol Device:R_Small
- added U11: W25Q128JV, Package_SO:SOIC-8_5.275x5.275mm_P1.27mm, symbol Memory_Flash:W25X40CLSN
Connections:
- net +3.3V: now also C60.1, R21.2, U11.3 (~{WP}), U11.7 (~{HOLD}), U11.8 (VCC)
- net GND: now also C60.2, R20.1, U11.4 (GND)
- net LED_DEBUG: now reaches U1.18 (PB0)
- net LED_DEBUG: now also D5.2 (A), D6.1 (K)
- net MEM_SCK: now reaches U1.21 (PB10)
- net MEM_SCK: now also U11.6 (SCK)
- net MEM_CS: now reaches U1.25 (PB12)
- net MEM_CS: now also U11.1 (~{CS})
- net MEM_MISO: now reaches U1.27 (PB14)
- net MEM_MISO: now also U11.2 (DO(IO1))
- net MEM_MOSI: now reaches U1.28 (PB15)
- net MEM_MOSI: now also U11.5 (DI(IO0))
- new net: D5.1 (K), R20.2
- new net: D6.2 (A), R21.1
Other:
- note added: "Debug LED"
- note added: "Flash Storage"
- moved on the sheet: J5
